File: SW-DUAL-10A.kicad_sch (KiCad schematic)
At the start: 26 parts, among them J1 SW1, J2 SW2, J3 GND +SW1, J4 GND +SW2, J5 GND +12V, U1 BTS7002-1EPP, U2 BTS7002-1EPP

Commit message: everything is on the layout, needs a lot of tuning
Parts:
- removed J3: GND +SW1, VP0265840000G, symbol SamacSys_Parts:VP0265840000G
- removed J4: GND +SW2, VP0265840000G, symbol SamacSys_Parts:VP0265840000G
- added J3, J4: Screw_Terminal_01x02, TerminalBlock_Phoenix:TerminalBlock_Phoenix_MKDS-1,5-2-5.08_1x02_P5.08mm_Horizontal, symbol Connector:Screw_Terminal_01x02
- J5: value GND +12V -> PWRIN
- R11, R12: footprint Resistor_SMD:R_0603_1608Metric_Pad0.98x0.95mm_HandSolder -> Resistor_THT:R_Axial_DIN0207_L6.3mm_D2.5mm_P7.62mm_Horizontal
- RGND1: renamed from R1; footprint Resistor_SMD:R_0805_2012Metric_Pad1.20x1.40mm_HandSolder -> Resistor_SMD:R_0603_1608Metric_Pad0.98x0.95mm_HandSolder
- RGND2: renamed from R2; footprint Resistor_SMD:R_0805_2012Metric_Pad1.20x1.40mm_HandSolder -> Resistor_SMD:R_0603_1608Metric_Pad0.98x0.95mm_HandSolder
Connections:
- net GND: now also J3.1 (Pin_1), J4.1 (Pin_1)
- net SW1OUT: now also J3.2 (Pin_2)
- net SW2OUT: now also J4.2 (Pin_2)

Commit message: updates
Parts:
- U1: footprint Package_SO:Infineon_PG-TSDSO-14-22 -> SamacSys_Parts:SOP65P600X115-15N
Changed lines of the file:
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@@
 			)
 		)
-		(property "Footprint" "Package_SO:Infineon_PG-TSDSO-14-22"
+		(property "Footprint" "SamacSys_Parts:SOP65P600X115-15N"
 			(at 114.3 74.93 0)
 			(effects

Commit message: added some mounting holes, pretty much finished, send it to the fab
Parts:
- added H1, H2, H3, H4: M4 4.3mm, MountingHole:MountingHole_4.3mm_M4, symbol Mechanical:MountingHole
- J3: value Screw_Terminal_01x02 -> Switch1
- J4: value Screw_Terminal_01x02 -> Switch2
- U2: footprint Package_SO:Infineon_PG-TSDSO-14-22 -> SamacSys_Parts:SOP65P600X115-15N
